Commit message: use package:// scheme to reference mesh files

File: model.urdf (robot description, URDF)
Before this commit: robot huboplus, 59 links, 58 joints
Links:
- link Body_Head: geometry collision mesh filename=package://hubo-urdf/meshes/Body_Head_col.dae; visual mesh filename=package://hubo-urdf/meshes/Body_Head_vis.dae
- link Body_Hip: geometry collision mesh filename=package://hubo-urdf/meshes/Body_Hip_col.dae; visual mesh filename=package://hubo-urdf/meshes/Body_Hip_vis.dae
- link Body_LAP: geometry collision mesh filename=package://hubo-urdf/meshes/Body_LAP_col.dae; visual mesh filename=package://hubo-urdf/meshes/Body_LAP_vis.dae
- link Body_LAR: geometry collision mesh filename=package://hubo-urdf/meshes/Body_LAR_col.dae; visual mesh filename=package://hubo-urdf/meshes/Body_LAR_vis.dae
- link Body_LEP: geometry collision mesh filename=package://hubo-urdf/meshes/Body_LEP_col.dae; visual mesh filename=package://hubo-urdf/meshes/Body_LEP_vis.dae
- link Body_LHP: geometry collision mesh filename=package://hubo-urdf/meshes/Body_LHP_col.dae; visual mesh filename=package://hubo-urdf/meshes/Body_LHP_vis.dae
- link Body_LHR: geometry collision mesh filename=package://hubo-urdf/meshes/Body_LHR_col.dae; visual mesh filename=package://hubo-urdf/meshes/Body_LHR_vis.dae
- link Body_LHY: geometry collision mesh filename=package://hubo-urdf/meshes/Body_LHY_col.dae; visual mesh filename=package://hubo-urdf/meshes/Body_LHY_vis.dae
- link Body_LKP: geometry collision mesh filename=package://hubo-urdf/meshes/Body_LKP_col.dae; visual mesh filename=package://hubo-urdf/meshes/Body_LKP_vis.dae
- link Body_LSP: geometry collision mesh filename=package://hubo-urdf/meshes/Body_LSP_col.dae; visual mesh filename=package://hubo-urdf/meshes/Body_LSP_vis.dae
- link Body_LSR: geometry collision mesh filename=package://hubo-urdf/meshes/Body_LSR_col.dae; visual mesh filename=package://hubo-urdf/meshes/Body_LSR_vis.dae
- link Body_LSY: geometry collision mesh filename=package://hubo-urdf/meshes/Body_LSY_col.dae; visual mesh filename=package://hubo-urdf/meshes/Body_LSY_vis.dae
- link Body_LWP: geometry collision mesh filename=package://hubo-urdf/meshes/Body_LWP_col.dae; visual mesh filename=package://hubo-urdf/meshes/Body_LWP_vis.dae
- link Body_LWY: geometry collision mesh filename=package://hubo-urdf/meshes/Body_LWY_col.dae; visual mesh filename=package://hubo-urdf/meshes/Body_LWY_vis.dae
- link Body_Neck: geometry collision mesh filename=package://hubo-urdf/meshes/Body_Neck_col.dae
- link Body_RAP: geometry collision mesh filename=package://hubo-urdf/meshes/Body_RAP_col.dae; visual mesh filename=package://hubo-urdf/meshes/Body_RAP_vis.dae
- link Body_RAR: geometry collision mesh filename=package://hubo-urdf/meshes/Body_RAR_col.dae; visual mesh filename=package://hubo-urdf/meshes/Body_RAR_vis.dae
- link Body_REP: geometry collision mesh filename=package://hubo-urdf/meshes/Body_REP_col.dae; visual mesh filename=package://hubo-urdf/meshes/Body_REP_vis.dae
- link Body_RHP: geometry collision mesh filename=package://hubo-urdf/meshes/Body_RHP_col.dae; visual mesh filename=package://hubo-urdf/meshes/Body_RHP_vis.dae
- link Body_RHR: geometry collision mesh filename=package://hubo-urdf/meshes/Body_RHR_col.dae; visual mesh filename=package://hubo-urdf/meshes/Body_RHR_vis.dae
- link Body_RHY: geometry collision mesh filename=package://hubo-urdf/meshes/Body_RHY_col.dae; visual mesh filename=package://hubo-urdf/meshes/Body_RHY_vis.dae
- link Body_RKP: geometry collision mesh filename=package://hubo-urdf/meshes/Body_RKP_col.dae; visual mesh filename=package://hubo-urdf/meshes/Body_RKP_vis.dae
- link Body_RSP: geometry collision mesh filename=package://hubo-urdf/meshes/Body_RSP_col.dae; visual mesh filename=package://hubo-urdf/meshes/Body_RSP_vis.dae
- link Body_RSR: geometry collision mesh filename=package://hubo-urdf/meshes/Body_RSR_col.dae; visual mesh filename=package://hubo-urdf/meshes/Body_RSR_vis.dae
- link Body_RSY: geometry collision mesh filename=package://hubo-urdf/meshes/Body_RSY_col.dae; visual mesh filename=package://hubo-urdf/meshes/Body_RSY_vis.dae
- link Body_RWP: geometry collision mesh filename=package://hubo-urdf/meshes/Body_RWP_col.dae; visual mesh filename=package://hubo-urdf/meshes/Body_RWP_vis.dae
- link Body_RWY: geometry collision mesh filename=package://hubo-urdf/meshes/Body_RWY_col.dae; visual mesh filename=package://hubo-urdf/meshes/Body_RWY_vis.dae
- link Body_Torso: geometry collision mesh filename=package://hubo-urdf/meshes/Body_Torso_col.dae; visual mesh filename=package://hubo-urdf/meshes/Body_Torso_vis.dae
- link leftIndexDistal: geometry collision mesh filename=package://hubo-urdf/meshes/leftIndexDistal_vis.dae; visual mesh filename=package://hubo-urdf/meshes/leftIndexDistal_vis.dae
- link leftIndexMedial: geometry collision mesh filename=package://hubo-urdf/meshes/leftIndexMedial_vis.dae; visual mesh filename=package://hubo-urdf/meshes/leftIndexMedial_vis.dae
- link leftIndexProximal: geometry collision mesh filename=package://hubo-urdf/meshes/leftIndexProximal_vis.dae; visual mesh filename=package://hubo-urdf/meshes/leftIndexProximal_vis.dae
- link leftMiddleDistal: geometry collision mesh filename=package://hubo-urdf/meshes/leftMiddleDistal_vis.dae; visual mesh filename=package://hubo-urdf/meshes/leftMiddleDistal_vis.dae
- link leftMiddleMedial: geometry collision mesh filename=package://hubo-urdf/meshes/leftMiddleMedial_vis.dae; visual mesh filename=package://hubo-urdf/meshes/leftMiddleMedial_vis.dae
- link leftMiddleProximal: geometry collision mesh filename=package://hubo-urdf/meshes/leftMiddleProximal_vis.dae; visual mesh filename=package://hubo-urdf/meshes/leftMiddleProximal_vis.dae
- link leftPinkyDistal: geometry collision mesh filename=package://hubo-urdf/meshes/leftPinkyDistal_vis.dae; visual mesh filename=package://hubo-urdf/meshes/leftPinkyDistal_vis.dae
- link leftPinkyMedial: geometry collision mesh filename=package://hubo-urdf/meshes/leftPinkyMedial_vis.dae; visual mesh filename=package://hubo-urdf/meshes/leftPinkyMedial_vis.dae
- link leftPinkyProximal: geometry collision mesh filename=package://hubo-urdf/meshes/leftPinkyProximal_vis.dae; visual mesh filename=package://hubo-urdf/meshes/leftPinkyProximal_vis.dae
- link leftRingDistal: geometry collision mesh filename=package://hubo-urdf/meshes/leftRingDistal_vis.dae; visual mesh filename=package://hubo-urdf/meshes/leftRingDistal_vis.dae
- link leftRingMedial: geometry collision mesh filename=package://hubo-urdf/meshes/leftRingMedial_vis.dae; visual mesh filename=package://hubo-urdf/meshes/leftRingMedial_vis.dae
- link leftRingProximal: geometry collision mesh filename=package://hubo-urdf/meshes/leftRingProximal_vis.dae; visual mesh filename=package://hubo-urdf/meshes/leftRingProximal_vis.dae
- link leftThumbDistal: geometry collision mesh filename=package://hubo-urdf/meshes/leftThumbDistal_vis.dae; visual mesh filename=package://hubo-urdf/meshes/leftThumbDistal_vis.dae
- link leftThumbMedial: geometry collision mesh filename=package://hubo-urdf/meshes/leftThumbMedial_vis.dae; visual mesh filename=package://hubo-urdf/meshes/leftThumbMedial_vis.dae
- link leftThumbProximal: geometry collision mesh filename=package://hubo-urdf/meshes/leftThumbProximal_vis.dae; visual mesh filename=package://hubo-urdf/meshes/leftThumbProximal_vis.dae
- link rightIndexDistal: geometry collision mesh filename=package://hubo-urdf/meshes/rightIndexDistal_vis.dae; visual mesh filename=package://hubo-urdf/meshes/rightIndexDistal_vis.dae
- link rightIndexMedial: geometry collision mesh filename=package://hubo-urdf/meshes/rightIndexMedial_vis.dae; visual mesh filename=package://hubo-urdf/meshes/rightIndexMedial_vis.dae
- link rightIndexProximal: geometry collision mesh filename=package://hubo-urdf/meshes/rightIndexProximal_vis.dae; visual mesh filename=package://hubo-urdf/meshes/rightIndexProximal_vis.dae
- link rightMiddleDistal: geometry collision mesh filename=package://hubo-urdf/meshes/rightMiddleDistal_vis.dae; visual mesh filename=package://hubo-urdf/meshes/rightMiddleDistal_vis.dae
- link rightMiddleMedial: geometry collision mesh filename=package://hubo-urdf/meshes/rightMiddleMedial_vis.dae; visual mesh filename=package://hubo-urdf/meshes/rightMiddleMedial_vis.dae
- link rightMiddleProximal: geometry collision mesh filename=package://hubo-urdf/meshes/rightMiddleProximal_vis.dae; visual mesh filename=package://hubo-urdf/meshes/rightMiddleProximal_vis.dae
- link rightPinkyDistal: geometry collision mesh filename=package://hubo-urdf/meshes/rightPinkyDistal_vis.dae; visual mesh filename=package://hubo-urdf/meshes/rightPinkyDistal_vis.dae
- link rightPinkyMedial: geometry collision mesh filename=package://hubo-urdf/meshes/rightPinkyMedial_vis.dae; visual mesh filename=package://hubo-urdf/meshes/rightPinkyMedial_vis.dae
- link rightPinkyProximal: geometry collision mesh filename=package://hubo-urdf/meshes/rightPinkyProximal_vis.dae; visual mesh filename=package://hubo-urdf/meshes/rightPinkyProximal_vis.dae
- link rightRingDistal: geometry collision mesh filename=package://hubo-urdf/meshes/rightRingDistal_vis.dae; visual mesh filename=package://hubo-urdf/meshes/rightRingDistal_vis.dae
- link rightRingMedial: geometry collision mesh filename=package://hubo-urdf/meshes/rightRingMedial_vis.dae; visual mesh filename=package://hubo-urdf/meshes/rightRingMedial_vis.dae
- link rightRingProximal: geometry collision mesh filename=package://hubo-urdf/meshes/rightRingProximal_vis.dae; visual mesh filename=package://hubo-urdf/meshes/rightRingProximal_vis.dae
- link rightThumbDistal: geometry collision mesh filename=package://hubo-urdf/meshes/rightThumbDistal_vis.dae; visual mesh filename=package://hubo-urdf/meshes/rightThumbDistal_vis.dae
- link rightThumbMedial: geometry collision mesh filename=package://hubo-urdf/meshes/rightThumbMedial_vis.dae; visual mesh filename=package://hubo-urdf/meshes/rightThumbMedial_vis.dae
- link rightThumbProximal: geometry collision mesh filename=package://hubo-urdf/meshes/rightThumbProximal_vis.dae; visual mesh filename=package://hubo-urdf/meshes/rightThumbProximal_vis.dae

Commit message: fix the robot model: don't let it loose its head in Gazebo
The robot seemed to be headless in the Gazebo simulator.
This was probably due to the physics simulation. Neck-related
links had zero mass. This probably leads to "infinite acceleration"
related effects.

Solution: set non-zero inertial parameters for neck-related links.

From Gazebo related tutorial:

    "For the Gazebo physics engine to work properly, the <inertial>
    element must be provided as documented on the URDF link element
    page. For links to not be ignored in Gazebo, their mass must be
    greater than zero. Additionally, links with zero principal
    moment of inertia (ixx, iyy, izz) could lead to infinite
    acceleration under any finite torque application."

see
http://gazebosim.org/wiki/Tutorials/1.9/Using_A_URDF_In_Gazebo#.3Cinertial.3E_Element

File: model.urdf (robot description, URDF)
Before this commit: robot huboplus, 59 links, 58 joints
Links:
- link Body_Head_Empty: mass None -> 1e-4
- link Body_Neck: mass None -> 1e-4

Commit message: make head-related joints that are not driven fixed
do not let the robot's head fall on side

File: model.urdf (robot description, URDF)
Before this commit: robot huboplus, 59 links, 58 joints
Joints:
- joint HNR: axis 1 0 0 -> (none); limit lower=-0.523599 upper=0.523599 effort=10.0 velocity=1.0 -> (none); type revolute -> fixed
- joint NKY: axis 0 0 1 -> (none); limit lower=-1.5 upper=1.5 effort=10.0 velocity=1.0 -> (none); type revolute -> fixed
